Commit message: Mount the wrist RealSense D415 and start the cameras on hardware
Port the x86 rig camera integration from wip/servoj-625hz-config onto
the IQ9 camera launch files already on main:

- fr5.xacro: mount the PickNik camera adapter bracket on tool0 and the
  wrist_mounted_camera D415 on it, from picknik_accessories.
- fr5.srdf: disable collisions between the bracket/D415 and the wrist
  links. Without these the planner reports the rigidly mounted camera
  as colliding with the wrist (the "red sphere").
- config.yaml / robot_drivers.launch.py: use robot_drivers.launch.py as
  the persist launch so rs_cameras.launch.xml (wrist + observer D415s)
  actually runs. Previously it pointed at blank.launch.py.
- package.xml: depend on picknik_accessories, realsense2_camera and
  realsense2_description.
- Add picknik_accessories as a pinned submodule instead of the copied
  files the wip branch carried, plus fanuc at the same SHA as its nested
  copy so rosdep resolves fanuc_lrmate200id_support (same layout as
  moveit_pro_kinova_ws).

Co-Authored-By: Claude Code <noreply@anthropic.com>

File: src/fairino_hw/description/fr5.xacro (robot description, xacro)
@@ -16,4 +16,26 @@
     <origin xyz="0 0 0.101" rpy="0 0 ${pi}" />
   </joint>
+  <!-- Wrist-mounted RealSense D415 on the PickNik UR-style camera adapter bracket,
+       used directly from the picknik_accessories package (same pattern as
+       picknik_ur_base_config's attachments macro). Parented to tool0 (the flange).
+       Bracket geometry is UR-designed, so the fit on the FR5 flange is nominal
+       (good for visualization + TF); swap the bracket or adjust origins for a real
+       Fairino mount. -->
+  <xacro:include
+    filename="$(find picknik_accessories)/descriptions/brackets/ur_realsense_camera_adapter/picknik_ur_camera_adapter.urdf.xacro" />
+  <xacro:include
+    filename="$(find picknik_accessories)/descriptions/sensors/realsense_d415.urdf.xacro" />
+  <xacro:ur_realsense_camera_adapter
+    prefix=""
+    parent="tool0"
+    child_tool="realsense_camera_adapter_tool0"
+    child_camera="d415_mount_link" />
+  <xacro:realsense_d415
+    parent="d415_mount_link"
+    name="wrist_mounted_camera"
+    use_nominal_extrinsics="true"
+    use_mesh="true">
+    <origin xyz="0 0 0" rpy="0 0 0" />
+  </xacro:realsense_d415>
   <!-- ros2_control configuration for Fairino hardware -->
   <ros2_control name="FairinoSystem" type="system">
